Commit message: Refactored some joint names in workcell description.

File: abb_irb4400_support/urdf/irb4400_macro.xacro (robot description, xacro)
@@ -5,14 +5,14 @@
 		<link name="${prefix}base_link">
 			<visual>
-      			<geometry>
-        			<mesh filename="package://abb_irb4400_support/meshes/irb4400/visual/base_link.stl" />
-      			</geometry>
-      			<material name="abb_orange">
-        			<color rgba="1 0.43 0 1" />
-      			</material>
-    		</visual>
- 			<collision>
-				<geometry>
-					<mesh filename="package://abb_irb4400_support/meshes/irb4400/collision/base_link.stl" />
+				<geometry>
+					<mesh filename="package://abb_irb4400_support/meshes/irb4400/visual/base_link.stl"/>
+				</geometry>
+				<material name="abb_orange">
+					<color rgba="1 0.43 0 1"/>
+				</material>
+			</visual>
+			<collision>
+				<geometry>
+					<mesh filename="package://abb_irb4400_support/meshes/irb4400/collision/base_link.stl"/>
 				</geometry>
 				<material name="yellow">
@@ -23,12 +23,12 @@
 		<link name="${prefix}link_1">
 			<visual>
-      			<geometry>
-        			<mesh filename="package://abb_irb4400_support/meshes/irb4400/visual/link_1.stl" />
-      			</geometry>
-      			<material name="abb_orange"/>
-    		</visual>
-			<collision>
-				<geometry>
-					<mesh filename="package://abb_irb4400_support/meshes/irb4400/collision/link_1.stl" />
+				<geometry>
+					<mesh filename="package://abb_irb4400_support/meshes/irb4400/visual/link_1.stl"/>
+				</geometry>
+				<material name="abb_orange"/>
+			</visual>
+			<collision>
+				<geometry>
+					<mesh filename="package://abb_irb4400_support/meshes/irb4400/collision/link_1.stl"/>
 				</geometry>
 				<material name="yellow"/>
@@ -36,13 +36,13 @@
 		</link>
 		<link name="${prefix}link_2">
-		    <visual>
-      			<geometry>
-        			<mesh filename="package://abb_irb4400_support/meshes/irb4400/visual/link_2.stl" />
-      			</geometry>
-      			<material name="abb_orange"/>
-    		</visual>
-			<collision>
-				<geometry>
-					<mesh filename="package://abb_irb4400_support/meshes/irb4400/collision/link_2.stl" />
+			<visual>
+				<geometry>
+					<mesh filename="package://abb_irb4400_support/meshes/irb4400/visual/link_2.stl"/>
+				</geometry>
+				<material name="abb_orange"/>
+			</visual>
+			<collision>
+				<geometry>
+					<mesh filename="package://abb_irb4400_support/meshes/irb4400/collision/link_2.stl"/>
 				</geometry>
 				<material name="yellow"/>
@@ -51,13 +51,12 @@
 		<link name="${prefix}link_3">
 			<visual>
-			  	<geometry>
-					<mesh
-				  	filename="package://abb_irb4400_support/meshes/irb4400/visual/link_3.stl" />
-			  	</geometry>
-			  	<material name="abb_orange"/>
-			</visual>
-			<collision>
-				<geometry>
-					<mesh filename="package://abb_irb4400_support/meshes/irb4400/collision/link_3.stl" />
+				<geometry>
+					<mesh filename="package://abb_irb4400_support/meshes/irb4400/visual/link_3.stl"/>
+				</geometry>
+				<material name="abb_orange"/>
+			</visual>
+			<collision>
+				<geometry>
+					<mesh filename="package://abb_irb4400_support/meshes/irb4400/collision/link_3.stl"/>
 				</geometry>
 				<material name="yellow"/>
@@ -66,13 +65,12 @@
 		<link name="${prefix}link_4">
 			<visual>
-				  <geometry>
-					<mesh
-					  filename="package://abb_irb4400_support/meshes/irb4400/visual/link_4.stl" />
-				  </geometry>
-				  <material name="abb_orange"/>
-			</visual>
-			<collision>
-				<geometry>
-					<mesh filename="package://abb_irb4400_support/meshes/irb4400/collision/link_4.stl" />
+				<geometry>
+					<mesh filename="package://abb_irb4400_support/meshes/irb4400/visual/link_4.stl"/>
+				</geometry>
+				<material name="abb_orange"/>
+			</visual>
+			<collision>
+				<geometry>
+					<mesh filename="package://abb_irb4400_support/meshes/irb4400/collision/link_4.stl"/>
 				</geometry>
 				<material name="yellow"/>
@@ -82,11 +80,11 @@
 			<visual>
 				<geometry>
-					<mesh filename="package://abb_irb4400_support/meshes/irb4400/visual/link_5.stl" />
-				</geometry>
-				<material name="abb_orange"/>
-			</visual>
-			<collision>
-				<geometry>
-					<mesh filename="package://abb_irb4400_support/meshes/irb4400/collision/link_5.stl" />
+					<mesh filename="package://abb_irb4400_support/meshes/irb4400/visual/link_5.stl"/>
+				</geometry>
+				<material name="abb_orange"/>
+			</visual>
+			<collision>
+				<geometry>
+					<mesh filename="package://abb_irb4400_support/meshes/irb4400/collision/link_5.stl"/>
 				</geometry>
 				<material name="yellow"/>
@@ -96,13 +94,13 @@
 			<visual>
 				<geometry>
-					<mesh filename="package://abb_irb4400_support/meshes/irb4400/visual/link_6.stl" />
+					<mesh filename="package://abb_irb4400_support/meshes/irb4400/visual/link_6.stl"/>
 				</geometry>
 				<material name="lt_black">
-          <color rgba="0.3 0.3 0.3 1"/>
-        </material>
-			</visual>
-			<collision>
-				<geometry>
-					<mesh filename="package://abb_irb4400_support/meshes/irb4400/collision/link_6.stl" />
+					<color rgba="0.3 0.3 0.3 1"/>
+				</material>
+			</visual>
+			<collision>
+				<geometry>
+					<mesh filename="package://abb_irb4400_support/meshes/irb4400/collision/link_6.stl"/>
 				</geometry>
 				<material name="yellow"/>
@@ -112,118 +110,118 @@
 		<!-- Parallelogram -->
 		<link name="${prefix}link_d1">
-          <visual>
-            <geometry>
-              <mesh filename="package://abb_irb4400_support/meshes/irb4400/visual/link_d1.stl"/>
-            </geometry>
-            <material name="abb_orange"/>
-          </visual>
-        </link>
-        <link name="${prefix}link_d2">
-          <visual>
-            <geometry>
-              <mesh filename="package://abb_irb4400_support/meshes/irb4400/visual/link_d2.stl"/>
-            </geometry>
-            <material name="abb_orange"/>
-          </visual>
-        </link>
-        <link name="${prefix}link_d3">
-          <visual>
-            <geometry>
-              <mesh filename="package://abb_irb4400_support/meshes/irb4400/visual/link_d3.stl"/>
-            </geometry>
-            <material name="abb_orange"/>
-          </visual>
-        </link>
-        <link name="${prefix}link_d4">
-          <visual>
-            <geometry>
-              <mesh filename="package://abb_irb4400_support/meshes/irb4400/visual/link_d4.stl"/>
-            </geometry>
-            <material name="abb_orange"/>
-          </visual>
-        </link>
+			<visual>
+				<geometry>
+					<mesh filename="package://abb_irb4400_support/meshes/irb4400/visual/link_d1.stl"/>
+				</geometry>
+				<material name="abb_orange"/>
+			</visual>
+		</link>
+		<link name="${prefix}link_d2">
+			<visual>
+				<geometry>
+					<mesh filename="package://abb_irb4400_support/meshes/irb4400/visual/link_d2.stl"/>
+				</geometry>
+				<material name="abb_orange"/>
+			</visual>
+		</link>
+		<link name="${prefix}link_d3">
+			<visual>
+				<geometry>
+					<mesh filename="package://abb_irb4400_support/meshes/irb4400/visual/link_d3.stl"/>
+				</geometry>
+				<material name="abb_orange"/>
+			</visual>
+		</link>
+		<link name="${prefix}link_d4">
+			<visual>
+				<geometry>
+					<mesh filename="package://abb_irb4400_support/meshes/irb4400/visual/link_d4.stl"/>
+				</geometry>
+				<material name="abb_orange"/>
+			</visual>
+		</link>
 		<!-- end of link list -->
 		<!-- joint list -->
 		<joint name="${prefix}joint_1" type="revolute">
-			<parent link="${prefix}base_link" />
-			<child link="${prefix}link_1" />
-			<origin xyz="0 0 0" rpy="0 0 0" />
-			<axis xyz="0 0 1" />
+			<parent link="${prefix}base_link"/>
+			<child link="${prefix}link_1"/>
+			<origin xyz="0 0 0" rpy="0 0 0"/>
+			<axis xyz="0 0 1"/>
 			<limit lower="-2.8798" upper="2.8798" effort="0" velocity="2.6180"/>
 		</joint>
 		<joint name="${prefix}joint_2" type="revolute">
-			<parent link="${prefix}link_1" />
-			<child link="${prefix}link_2" />
-			<origin xyz="0.200 0 0.680" rpy="0 0 0" />
-			<axis xyz="0 1 0" />
-			<limit lower="-1.2217" upper="1.6755" effort="0" velocity="2.0944"/>
-  		</joint>
+			<parent link="${prefix}link_1"/>
+			<child link="${prefix}link_2"/>
+			<origin xyz="0.200 0 0.680" rpy="0 0 0"/>
+			<axis xyz="0 1 0"/>
+			<limit lower="-1.2217" upper="1.6755" effort="0" velocity="2.0944"/>
+		</joint>
 		<joint name="${prefix}joint_3" type="revolute">
-			<parent link="${prefix}link_2" />
-			<child link="${prefix}link_3" />
-			<origin xyz="0 0 0.890" rpy="0 0 0" />
-			<axis xyz="0 1 0" />
+			<parent link="${prefix}link_2"/>
+			<child link="${prefix}link_3"/>
+			<origin xyz="0 0 0.890" rpy="0 0 0"/>
+			<axis xyz="0 1 0"/>
 			<limit lower="-1.0472" upper="1.1345" effort="0" velocity="2.0944"/>
 		</joint>
 		<joint name="${prefix}joint_4" type="revolute">
-			<parent link="${prefix}link_3" />
-			<child link="${prefix}link_4" />
-			<origin xyz="0 0 0.150" rpy="0 0 0" />
-			<axis xyz="1 0 0" />
+			<parent link="${prefix}link_3"/>
+			<child link="${prefix}link_4"/>
+			<origin xyz="0 0 0.150" rpy="0 0 0"/>
+			<axis xyz="1 0 0"/>
 			<limit lower="-3.4907" upper="3.4907" effort="0" velocity="3.9270"/>
 		</joint>
 		<joint name="${prefix}joint_5" type="revolute">
-			<parent link="${prefix}link_4" />
-			<child link="${prefix}link_5" />
-			<origin xyz="0.880 0 0" rpy="0 0 0" />
-			<axis xyz="0 1 0" />
+			<parent link="${prefix}link_4"/>
+			<child link="${prefix}link_5"/>
+			<origin xyz="0.880 0 0" rpy="0 0 0"/>
+			<axis xyz="0 1 0"/>
 			<limit lower="-2.0944" upper="2.0944" effort="0" velocity="2.3633"/>
 		</joint>
 		<joint name="${prefix}joint_6" type="revolute">
-			<parent link="${prefix}link_5" />
-			<child link="${prefix}link_6" />
-			<origin xyz="0 0 0" rpy="0 0 0" />
-			<axis xyz="1 0 0" />
+			<parent link="${prefix}link_5"/>
+			<child link="${prefix}link_6"/>
+			<origin xyz="0 0 0" rpy="0 0 0"/>
+			<axis xyz="1 0 0"/>
 			<limit lower="-6.9813" upper="6.9813" effort="0" velocity="5.7596"/>
 		</joint>
-		<joint name="${prefix}joint_6-tool0" type="fixed">
+		<joint name="${prefix}tool0" type="fixed">
 			<parent link="${prefix}link_6"/>
 			<child link="${prefix}tool0"/>
-			<origin xyz="0.140 0 0" rpy="0 1.5708 0" />
-		</joint>
-      <!-- Parallelogram -->
-      <joint name="${prefix}joint_d1" type="revolute">
-        <parent link="${prefix}link_3"/>
-        <child link="${prefix}link_d1"/>
-        <origin xyz="-0.300 0 0" rpy="0 0 0"/>
-        <axis xyz="0 1 0"/>
-        <mimic joint="${prefix}joint_3" multiplier="-1.0" offset="0.0" />
-        <limit lower="-1.2217" upper="1.6755" effort="0" velocity="2.0944"/>
-      </joint>
-      <joint name="${prefix}joint_d2" type="revolute">
-        <parent link="${prefix}link_1"/>
-        <child link="${prefix}link_d2"/>
-        <origin xyz="0.200 0 0.680" rpy="0 0 0"/>
-        <axis xyz="0 1 0"/>
-        <mimic joint="${prefix}joint_2" multiplier="1.0" offset="0.0" />
-        <mimic joint="${prefix}joint_3" multiplier="1.0" offset="0.0" />
-        <limit lower="-1.2217" upper="1.6755" effort="0" velocity="2.0944"/>
-      </joint>
-      <joint name="${prefix}joint_d3" type="fixed">
-        <parent link="${prefix}link_1"/>
-        <child link="${prefix}link_d3"/>
-        <origin xyz="0 0 0" rpy="0 0 0"/>
-        <axis xyz="0 1 0"/>
-        <mimic joint="${prefix}joint_2" multiplier="0.5" offset="0.0" />
-        <limit lower="-1.2217" upper="1.6755" effort="0" velocity="2.0944"/>
-      </joint>
-      <joint name="${prefix}joint_d4" type="fixed">
-        <parent link="${prefix}link_1"/>
-        <child link="${prefix}link_d4"/>
-        <origin xyz="0 0 0" rpy="0 0 0"/>
-        <axis xyz="0 1 0"/>
-        <mimic joint="${prefix}joint_2" multiplier="0.5" offset="0.0" />
-        <limit lower="-1.2217" upper="1.6755" effort="0" velocity="2.0944"/>
-      </joint>
+			<origin xyz="0.140 0 0" rpy="0 1.5708 0"/>
+		</joint>
+		<!-- Parallelogram -->
+		<joint name="${prefix}joint_d1" type="revolute">
+			<parent link="${prefix}link_3"/>
+			<child link="${prefix}link_d1"/>
+			<origin xyz="-0.300 0 0" rpy="0 0 0"/>
+			<axis xyz="0 1 0"/>
+			<mimic joint="${prefix}joint_3" multiplier="-1.0" offset="0.0"/>
+			<limit lower="-1.2217" upper="1.6755" effort="0" velocity="2.0944"/>
+		</joint>
+		<joint name="${prefix}joint_d2" type="revolute">
+			<parent link="${prefix}link_1"/>
+			<child link="${prefix}link_d2"/>
+			<origin xyz="0.200 0 0.680" rpy="0 0 0"/>
+			<axis xyz="0 1 0"/>
+			<mimic joint="${prefix}joint_2" multiplier="1.0" offset="0.0"/>
+			<mimic joint="${prefix}joint_3" multiplier="1.0" offset="0.0"/>
+			<limit lower="-1.2217" upper="1.6755" effort="0" velocity="2.0944"/>
+		</joint>
+		<joint name="${prefix}joint_d3" type="fixed">
+			<parent link="${prefix}link_1"/>
+			<child link="${prefix}link_d3"/>
+			<origin xyz="0 0 0" rpy="0 0 0"/>
+			<axis xyz="0 1 0"/>
+			<mimic joint="${prefix}joint_2" multiplier="0.5" offset="0.0"/>
+			<limit lower="-1.2217" upper="1.6755" effort="0" velocity="2.0944"/>
+		</joint>
+		<joint name="${prefix}joint_d4" type="fixed">
+			<parent link="${prefix}link_1"/>
+			<child link="${prefix}link_d4"/>
+			<origin xyz="0 0 0" rpy="0 0 0"/>
+			<axis xyz="0 1 0"/>
+			<mimic joint="${prefix}joint_2" multiplier="0.5" offset="0.0"/>
+			<limit lower="-1.2217" upper="1.6755" effort="0" velocity="2.0944"/>
+		</joint>
 		<!-- end of joint list -->
 	</xacro:macro>

File: aimen_workcell/urdf/abb_robot.xacro (robot description, xacro)
@@ -1,35 +1,19 @@
 <?xml version="1.0" ?>
 <robot name="abb_robot" xmlns:xacro="http://ros.org/wiki/xacro">
-  <property name="pi" value="3.141592654" />
-  <!-- Robot -->
-  <xacro:include filename="$(find abb_irb4400_support)/urdf/irb4400_macro.xacro"/>
-  <xacro:abb_irb4400 prefix=""/>
-  <joint name="world-irb4400" type="fixed">
-    <parent link="world"/>
-    <child link="base_link"/>
-    <origin xyz="0 0 0.067" rpy="0 0 0" />
-  </joint>
-  <!-- Table -->
-  <xacro:include filename="$(find aimen_workcell)/urdf/irbp_a250.xacro"/>
-  <joint name="world-irbp_a250/base_link" type="fixed">
-    <parent link="world"/>
-    <child link="irbp_a250/base_link"/>
-    <origin xyz="1.753 0.015 -0.003" rpy="-0.005599 -0.005742 1.550718" />
-  </joint>
-  <link name="table0">
-    <visual>
-    <geometry>
-      <mesh filename="package://aimen_workcell/meshes/table/table.stl"/>
-    </geometry>
-    <material name="gray">
-      <color rgba="0.4 0.4 0.4 0.6"/>
-    </material>
-  </visual>
-  </link>
-  <joint name="tool0-table0" type="fixed">
-    <parent link="irbp_a250/tool0"/>
-    <child link="table0"/>
-    <origin xyz="0 0 0" rpy="0 0 0" />
-    <axis xyz="0 0 1"/>
-  </joint>
+    <property name="pi" value="3.141592654"/>
+    <!-- Robot -->
+    <xacro:include filename="$(find abb_irb4400_support)/urdf/irb4400_macro.xacro"/>
+    <xacro:abb_irb4400 prefix=""/>
+    <joint name="irb4400" type="fixed">
+        <parent link="world"/>
+        <child link="base_link"/>
+        <origin xyz="0 0 0.067" rpy="0 0 0"/>
+    </joint>
+    <!-- Robot table -->
+    <xacro:include filename="$(find aimen_workcell)/urdf/irbp_a250.xacro"/>
+    <joint name="irbp_a250" type="fixed">
+        <parent link="world"/>
+        <child link="irbp_a250/base_link"/>
+        <origin xyz="1.753 0.015 -0.003" rpy="-0.005599 -0.005742 1.550718"/>
+    </joint>
 </robot>

File: aimen_workcell/urdf/irbp_a250.xacro (robot description, xacro)
@@ -107,5 +107,5 @@
     <limit effort="100" velocity="3.1416" />
   </joint>
-  <joint name="${name}joint4-tool0" type="fixed">
+  <joint name="${name}tool0" type="fixed">
     <parent link="${name}link_4" />
     <child link="${name}tool0" />

File: aimen_workcell/urdf/workcell.xacro (robot description, xacro)
@@ -1,29 +1,46 @@
 <?xml version="1.0" ?>
 <robot name="aimen_workcell" xmlns:xacro="http://ros.org/wiki/xacro">
-  <property name="pi" value="3.141592654" />
-  <link name="world" />
-  <!-- Robot -->
-  <xacro:include filename="$(find aimen_workcell)/urdf/abb_robot.xacro"/>
-  <joint name="world-abb_robot" type="fixed">
-    <parent link="world"/>
-    <child link="base_link"/>
-    <origin xyz="0 0 0.067" rpy="0 0 0" />
-  </joint>
-  <!-- Cell walls -->
-  <link name="walls">
-  <visual>
-    <geometry>
-      <mesh filename="package://aimen_workcell/meshes/cell/cell.stl"/>
-    </geometry>
-    <origin xyz="0 0 0" />
-    <material name="white">
-      <color rgba="1 1 1 0.75"/>
-    </material>
-  </visual>
-  </link>
-  <joint name="world_to_walls" type="fixed">
-    <parent link="world" />
-    <child link="walls" />
-    <origin xyz="0 0 0" />
-  </joint>
+    <property name="pi" value="3.141592654"/>
+    <link name="world"/>
+    <!-- Robot -->
+    <xacro:include filename="$(find aimen_workcell)/urdf/abb_robot.xacro"/>
+    <joint name="abb_robot" type="fixed">
+        <parent link="world"/>
+        <child link="base_link"/>
+        <origin xyz="0 0 0.067" rpy="0 0 0"/>
+    </joint>
+    <!-- Table -->
+    <link name="table0">
+        <visual>
+            <geometry>
+                <mesh filename="package://aimen_workcell/meshes/table/table.stl"/>
+            </geometry>
+            <material name="gray">
+                <color rgba="0.4 0.4 0.4 0.6"/>
+            </material>
+        </visual>
+    </link>
+    <joint name="table0" type="fixed">
+        <parent link="irbp_a250/tool0"/>
+        <child link="table0"/>
+        <origin xyz="0 0 0" rpy="0 0 0"/>
+        <axis xyz="0 0 1"/>
+    </joint>
+    <!-- Cell walls -->
+    <link name="walls">
+        <visual>
+            <geometry>
+                <mesh filename="package://aimen_workcell/meshes/cell/cell.stl"/>
+            </geometry>
+            <origin xyz="0 0 0"/>
+            <material name="white">
+                <color rgba="1 1 1 0.75"/>
+            </material>
+        </visual>
+    </link>
+    <joint name="walls" type="fixed">
+        <parent link="world"/>
+        <child link="walls"/>
+        <origin xyz="0 0 0"/>
+    </joint>
 </robot>
