Commit message: AAdded aimen_driver from proper_abb package.

File: aimen_abb/urdf/irb4400.urdf (robot description, URDF)
Before this commit: robot abb_irb4400, 9 links, 8 joints
Links:
- link base_link: geometry collision mesh filename=package://aimen_abb/meshes/irb4400/collision/base_link.stl; visual mesh filename=package://aimen_abb/meshes/irb4400/visual/base_link.stl
- link link_1: geometry collision mesh filename=package://aimen_abb/meshes/irb4400/collision/link_1.stl; visual mesh filename=package://aimen_abb/meshes/irb4400/visual/link_1.stl
- link link_2: geometry collision mesh filename=package://aimen_abb/meshes/irb4400/collision/link_2.stl; visual mesh filename=package://aimen_abb/meshes/irb4400/visual/link_2.stl
- link link_3: geometry collision mesh filename=package://aimen_abb/meshes/irb4400/collision/link_3.stl; visual mesh filename=package://aimen_abb/meshes/irb4400/visual/link_3.stl
- link link_4: geometry collision mesh filename=package://aimen_abb/meshes/irb4400/collision/link_4.stl; visual mesh filename=package://aimen_abb/meshes/irb4400/visual/link_4.stl
- link link_5: geometry collision mesh filename=package://aimen_abb/meshes/irb4400/collision/link_5.stl; visual mesh filename=package://aimen_abb/meshes/irb4400/visual/link_5.stl
- link link_6: geometry collision mesh filename=package://aimen_abb/meshes/irb4400/collision/link_6.stl; visual mesh filename=package://aimen_abb/meshes/irb4400/visual/link_6.stl
- link link_d2: geometry visual mesh filename=package://aimen_abb/meshes/irb4400/visual/link_d2.stl

File: aimen_abb/urdf/irb4400.xacro (robot description, xacro)
@@ -1,5 +1,5 @@
 <?xml version="1.0" ?>
 <robot name="abb_irb4400" xmlns:xacro="http://ros.org/wiki/xacro">
-  <xacro:include filename="$(find abb_irb4400_support)/urdf/irb4400_macro.xacro"/>
+  <xacro:include filename="$(find aimen_abb)/urdf/irb4400_macro.xacro"/>
   <xacro:abb_irb4400 prefix=""/>
 </robot>

File: aimen_abb/urdf/irb4400_macro.xacro (robot description, xacro)
@@ -6,5 +6,5 @@
 			<visual>
 				<geometry>
-					<mesh filename="package://abb_irb4400_support/meshes/irb4400/visual/base_link.stl"/>
+					<mesh filename="package://aimen_abb/meshes/irb4400/visual/base_link.stl"/>
 				</geometry>
 				<material name="abb_orange">
@@ -14,5 +14,5 @@
 			<collision>
 				<geometry>
-					<mesh filename="package://abb_irb4400_support/meshes/irb4400/collision/base_link.stl"/>
+					<mesh filename="package://aimen_abb/meshes/irb4400/collision/base_link.stl"/>
 				</geometry>
 				<material name="yellow">
@@ -24,11 +24,11 @@
 			<visual>
 				<geometry>
-					<mesh filename="package://abb_irb4400_support/meshes/irb4400/visual/link_1.stl"/>
-				</geometry>
-				<material name="abb_orange"/>
-			</visual>
-			<collision>
-				<geometry>
-					<mesh filename="package://abb_irb4400_support/meshes/irb4400/collision/link_1.stl"/>
+					<mesh filename="package://aimen_abb/meshes/irb4400/visual/link_1.stl"/>
+				</geometry>
+				<material name="abb_orange"/>
+			</visual>
+			<collision>
+				<geometry>
+					<mesh filename="package://aimen_abb/meshes/irb4400/collision/link_1.stl"/>
 				</geometry>
 				<material name="yellow"/>
@@ -38,11 +38,11 @@
 			<visual>
 				<geometry>
-					<mesh filename="package://abb_irb4400_support/meshes/irb4400/visual/link_2.stl"/>
-				</geometry>
-				<material name="abb_orange"/>
-			</visual>
-			<collision>
-				<geometry>
-					<mesh filename="package://abb_irb4400_support/meshes/irb4400/collision/link_2.stl"/>
+					<mesh filename="package://aimen_abb/meshes/irb4400/visual/link_2.stl"/>
+				</geometry>
+				<material name="abb_orange"/>
+			</visual>
+			<collision>
+				<geometry>
+					<mesh filename="package://aimen_abb/meshes/irb4400/collision/link_2.stl"/>
 				</geometry>
 				<material name="yellow"/>
@@ -52,11 +52,11 @@
 			<visual>
 				<geometry>
-					<mesh filename="package://abb_irb4400_support/meshes/irb4400/visual/link_3.stl"/>
-				</geometry>
-				<material name="abb_orange"/>
-			</visual>
-			<collision>
-				<geometry>
-					<mesh filename="package://abb_irb4400_support/meshes/irb4400/collision/link_3.stl"/>
+					<mesh filename="package://aimen_abb/meshes/irb4400/visual/link_3.stl"/>
+				</geometry>
+				<material name="abb_orange"/>
+			</visual>
+			<collision>
+				<geometry>
+					<mesh filename="package://aimen_abb/meshes/irb4400/collision/link_3.stl"/>
 				</geometry>
 				<material name="yellow"/>
@@ -66,11 +66,11 @@
 			<visual>
 				<geometry>
-					<mesh filename="package://abb_irb4400_support/meshes/irb4400/visual/link_4.stl"/>
-				</geometry>
-				<material name="abb_orange"/>
-			</visual>
-			<collision>
-				<geometry>
-					<mesh filename="package://abb_irb4400_support/meshes/irb4400/collision/link_4.stl"/>
+					<mesh filename="package://aimen_abb/meshes/irb4400/visual/link_4.stl"/>
+				</geometry>
+				<material name="abb_orange"/>
+			</visual>
+			<collision>
+				<geometry>
+					<mesh filename="package://aimen_abb/meshes/irb4400/collision/link_4.stl"/>
 				</geometry>
 				<material name="yellow"/>
@@ -80,11 +80,11 @@
 			<visual>
 				<geometry>
-					<mesh filename="package://abb_irb4400_support/meshes/irb4400/visual/link_5.stl"/>
-				</geometry>
-				<material name="abb_orange"/>
-			</visual>
-			<collision>
-				<geometry>
-					<mesh filename="package://abb_irb4400_support/meshes/irb4400/collision/link_5.stl"/>
+					<mesh filename="package://aimen_abb/meshes/irb4400/visual/link_5.stl"/>
+				</geometry>
+				<material name="abb_orange"/>
+			</visual>
+			<collision>
+				<geometry>
+					<mesh filename="package://aimen_abb/meshes/irb4400/collision/link_5.stl"/>
 				</geometry>
 				<material name="yellow"/>
@@ -94,5 +94,5 @@
 			<visual>
 				<geometry>
-					<mesh filename="package://abb_irb4400_support/meshes/irb4400/visual/link_6.stl"/>
+					<mesh filename="package://aimen_abb/meshes/irb4400/visual/link_6.stl"/>
 				</geometry>
 				<material name="lt_black">
@@ -102,5 +102,5 @@
 			<collision>
 				<geometry>
-					<mesh filename="package://abb_irb4400_support/meshes/irb4400/collision/link_6.stl"/>
+					<mesh filename="package://aimen_abb/meshes/irb4400/collision/link_6.stl"/>
 				</geometry>
 				<material name="yellow"/>
@@ -112,5 +112,5 @@
 			<visual>
 				<geometry>
-					<mesh filename="package://abb_irb4400_support/meshes/irb4400/visual/link_d1.stl"/>
+					<mesh filename="package://aimen_abb/meshes/irb4400/visual/link_d1.stl"/>
 				</geometry>
 				<material name="abb_orange"/>
@@ -120,5 +120,5 @@
 			<visual>
 				<geometry>
-					<mesh filename="package://abb_irb4400_support/meshes/irb4400/visual/link_d2.stl"/>
+					<mesh filename="package://aimen_abb/meshes/irb4400/visual/link_d2.stl"/>
 				</geometry>
 				<material name="abb_orange"/>
@@ -128,5 +128,5 @@
 			<visual>
 				<geometry>
-					<mesh filename="package://abb_irb4400_support/meshes/irb4400/visual/link_d3.stl"/>
+					<mesh filename="package://aimen_abb/meshes/irb4400/visual/link_d3.stl"/>
 				</geometry>
 				<material name="abb_orange"/>
@@ -136,5 +136,5 @@
 			<visual>
 				<geometry>
-					<mesh filename="package://abb_irb4400_support/meshes/irb4400/visual/link_d4.stl"/>
+					<mesh filename="package://aimen_abb/meshes/irb4400/visual/link_d4.stl"/>
 				</geometry>
 				<material name="abb_orange"/>

File: aimen_workcell/urdf/abb_robot.xacro (robot description, xacro)
@@ -3,5 +3,5 @@
     <property name="pi" value="3.141592654"/>
     <!-- Robot -->
-    <xacro:include filename="$(find abb_irb4400_support)/urdf/irb4400_macro.xacro"/>
+    <xacro:include filename="$(find aimen_abb)/urdf/irb4400_macro.xacro"/>
     <xacro:abb_irb4400 prefix=""/>
     <joint name="irb4400" type="fixed">
