Commit message: Fixed some issues in irbp model.

File: aimen_workcell/urdf/irbp_a250.xacro (robot description, xacro)
@@ -87,5 +87,5 @@
     <axis xyz="0 0 1" />
   </joint>
-  <joint name="${name}joint2" type="revolute">
+  <joint name="${name}joint2" type="fixed"><!--"revolute"-->
     <parent link="${name}link_1" />
     <child link="${name}link_2" />
@@ -100,5 +100,5 @@
     <axis xyz="0 1 0" />
   </joint>
-  <joint name="${name}joint4" type="continuous">
+  <joint name="${name}joint4" type="fixed"><!--"continuous"-->
     <parent link="${name}link_3" />
     <child link="${name}link_4" />

Commit message: Added joints state monitoring for irbpa250.

File: aimen_workcell/urdf/irbp_a250.xacro (robot description, xacro)
@@ -87,5 +87,5 @@
     <axis xyz="0 0 1" />
   </joint>
-  <joint name="${name}joint2" type="fixed"><!--"revolute"-->
+  <joint name="${name}joint2" type="revolute">
     <parent link="${name}link_1" />
     <child link="${name}link_2" />
@@ -100,5 +100,5 @@
     <axis xyz="0 1 0" />
   </joint>
-  <joint name="${name}joint4" type="fixed"><!--"continuous"-->
+  <joint name="${name}joint4" type="continuous">
     <parent link="${name}link_3" />
     <child link="${name}link_4" />
