Commit message: Kuka kr-210-2 robot model added

File: aimen_workcell/urdf/workcell.xacro (robot description, xacro)
@@ -4,6 +4,6 @@
     <link name="world"/>
     <!-- Robot -->
-    <xacro:include filename="$(find aimen_workcell)/urdf/abb_robot.xacro"/>
-    <joint name="abb_robot" type="fixed">
+    <xacro:include filename="$(find aimen_workcell)/urdf/abb_robot.xacro"/> <!-- kuka_robot -->
+    <joint name="abb_robot" type="fixed"> <!-- kuka_robot -->
         <parent link="world"/>
         <child link="base_link"/>
