Commit message: Kuka robot logger interface

File: aimen_workcell/urdf/kuka_robot.xacro (robot description, xacro)
@@ -3,7 +3,7 @@
     <property name="pi" value="3.141592654"/>
     <!-- Robot -->
-    <xacro:include filename="$(find aimen_kuka)/urdf/kr2102_macro.xacro"/>
-    <xacro:kuka_kr2102 prefix=""/>
-    <joint name="kr2102" type="fixed">
+    <xacro:include filename="$(find aimen_kuka)/urdf/kr1502_macro.xacro"/>
+    <xacro:kuka_kr1502 prefix=""/>
+    <joint name="kr1502" type="fixed">
         <parent link="world"/>
         <child link="base_link"/>
